Commit message: v3

File: description/ros2_control.xacro (robot description, xacro)
@@ -2,5 +2,5 @@
 <robot xmlns:xacro="http://www.ros.org/wiki/xacro">
     <xacro:unless value="$(arg sim_mode)">
-        <ros2_control name="RealRobot" type="system">
+        <ros2_control name="RealRobotFront" type="system">
             <hardware>
                 <plugin>diffdrive_arduino/DiffDriveArduino</plugin>
@@ -9,14 +9,4 @@
                 <param name="loop_rate">30</param>
                 <param name="device">/dev/ttyACM0</param>
-                <param name="baud_rate">57600</param>
-                <param name="timeout">1000</param>
-                <param name="enc_counts_per_rev">3436</param>
-            </hardware>
-            <hardware>
-                <plugin>diffdrive_arduino/DiffDriveArduino</plugin>
-                <param name="left_wheel_name">rear_left_wheel_joint</param>
-                <param name="right_wheel_name">rear_right_wheel_joint</param>
-                <param name="loop_rate">30</param>
-                <param name="device">/dev/ttyACM1</param>
                 <param name="baud_rate">57600</param>
                 <param name="timeout">1000</param>
@@ -39,5 +29,17 @@
                 <state_interface name="position"/>
             </joint>
-             <joint name="rear_left_wheel_joint">
+        </ros2_control>
+        <ros2_control name="RealRobotRear" type="system">
+            <hardware>
+                <plugin>diffdrive_arduino/DiffDriveArduino</plugin>
+                <param name="left_wheel_name">rear_left_wheel_joint</param>
+                <param name="right_wheel_name">rear_right_wheel_joint</param>
+                <param name="loop_rate">30</param>
+                <param name="device">/dev/ttyACM1</param>
+                <param name="baud_rate">57600</param>
+                <param name="timeout">1000</param>
+                <param name="enc_counts_per_rev">3436</param>
+            </hardware>
+            <joint name="rear_left_wheel_joint">
                 <command_interface name="velocity">
                     <param name="min">-10</param>
